File: hardware/rearbox/fused_output.kicad_sch (KiCad schematic)
At the start: 13 parts, among them U7 VND7020AJTR

Commit message: Changed power section
Parts:
- renumbered D1 to D3, D1 to D4
Changed lines of the file:
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@@
 (kicad_sch
-	(version 20231120)
+	(version 20250114)
 	(generator "eeschema")
-	(generator_version "8.0")
+	(generator_version "9.0")
 	(paper "A4")
 	(title_block
@@
 		(comment 1 "Reviewer:")
 	)
+	(text "GND"
+		(exclude_from_sim no)
+		(at 225.298 100.076 0)
+		(effects
+			(font
+				(size 1.27 1.27)
+			)
+			(justify left bottom)
+		)
+	)
+	(text "Auto-restart Mode"
+		(exclude_from_sim no)
+		(at 99.06 110.49 0)
+		(effects
+			(font
+				(size 1.27 1.27)
+			)
+			(justify left bottom)
+		)
+	)
+	(text "GND"
+		(exclude_from_sim no)
+		(at 225.298 122.936 0)
+		(effects
+			(font
+				(size 1.27 1.27)
+			)
+			(justify left bottom)
+		)
+	)
+	(text "Load"
+		(exclude_from_sim no)
+		(at 227.965 92.456 90)
+		(effects
+			(font
+				(size 1.27 1.27)
+			)
+			(justify left bottom)
+		)
+	)
+	(text "Load"
+		(exclude_from_sim no)
+		(at 227.965 115.316 90)
+		(effects
+			(font
+				(size 1.27 1.27)
+			)
+			(justify left bottom)
+		)
+	)
 	(junction
 		(at 205.74 85.09)
@@
 		)
 	)
-	(text "GND"
-		(exclude_from_sim no)
-		(at 225.298 100.076 0)
+	(label "OUT2"
+		(at 201.93 107.95 180)
 		(effects
 			(font
 				(size 1.27 1.27)
 			)
-			(justify left bottom)
-		)
-	)
-	(text "Auto-restart Mode"
-		(exclude_from_sim no)
-		(at 99.06 110.49 0)
+			(justify right bottom)
+		)
+	)
+	(label "OUT2"
+		(at 152.4 87.63 0)
 		(effects
 			(font
@@
 		)
 	)
-	(text "GND"
-		(exclude_from_sim no)
-		(at 225.298 122.936 0)
+	(label "OUT1"
+		(at 152.4 85.09 0)
 		(effects
 			(font
@@
 		)
 	)
-	(text "Load"
-		(exclude_from_sim no)
-		(at 227.965 92.456 90)
+	(label "OUT1"
+		(at 201.93 85.09 180)
 		(effects
 			(font
 				(size 1.27 1.27)
 			)
-			(justify left bottom)
-		)
-	)
-	(text "Load"
-		(exclude_from_sim no)
-		(at 227.965 115.316 90)
+			(justify right bottom)
+		)
+	)
+	(hierarchical_label "SE1"
+		(shape input)
+		(at 109.22 96.52 180)
 		(effects
 			(font
 				(size 1.27 1.27)
 			)
-			(justify left bottom)
-		)
-	)
-	(label "OUT2"
-		(at 201.93 107.95 180)
-		(fields_autoplaced yes)
+			(justify right)
+		)
+	)
+	(hierarchical_label "OUT2"
+		(shape output)
+		(at 213.36 107.95 0)
 		(effects
 			(font
 				(size 1.27 1.27)
 			)
-			(justify right bottom)
-		)
-	)
-	(label "OUT2"
-		(at 152.4 87.63 0)
-		(fields_autoplaced yes)
+			(justify left)
+		)
+	)
+	(hierarchical_label "SE"
+		(shape input)
+		(at 109.22 91.44 180)
 		(effects
 			(font
 				(size 1.27 1.27)
 			)
-			(justify left bottom)
-		)
-	)
-	(label "OUT1"
-		(at 152.4 85.09 0)
-		(fields_autoplaced yes)
+			(justify right)
+		)
+	)
+	(hierarchical_label "SENSE"
+		(shape output)
+		(at 167.64 102.87 0)
 		(effects
 			(font
 				(size 1.27 1.27)
 			)
-			(justify left bottom)
-		)
-	)
-	(label "OUT1"
-		(at 201.93 85.09 180)
-		(fields_autoplaced yes)
+			(justify left)
+		)
+	)
+	(hierarchical_label "OUT1"
+		(shape output)
+		(at 213.36 85.09 0)
 		(effects
 			(font
 				(size 1.27 1.27)
 			)
-			(justify right bottom)
-		)
-	)
-	(hierarchical_label "SE1"
+			(justify left)
+		)
+	)
+	(hierarchical_label "IN1"
 		(shape input)
-		(at 109.22 96.52 180)
-		(fields_autoplaced yes)
+		(at 109.22 85.09 180)
 		(effects
 			(font
@@
 		)
 	)
-	(hierarchical_label "OUT2"
-		(shape output)
-		(at 213.36 107.95 0)
-		(fields_autoplaced yes)
+	(hierarchical_label "IN2"
+		(shape input)
+		(at 109.22 87.63 180)
 		(effects
 			(font
 				(size 1.27 1.27)
 			)
-			(justify left)
-		)
-	)
-	(hierarchical_label "SE"
-		(shape input)
-		(at 109.22 91.44 180)
-		(fields_autoplaced yes)
-		(effects
-			(font
-				(size 1.27 1.27)
-			)
-			(justify right)
-		)
-	)
-	(hierarchical_label "SENSE"
-		(shape output)
-		(at 167.64 102.87 0)
-		(fields_autoplaced yes)
-		(effects
-			(font
-				(size 1.27 1.27)
-			)
-			(justify left)
-		)
-	)
-	(hierarchical_label "OUT1"
-		(shape output)
-		(at 213.36 85.09 0)
-		(fields_autoplaced yes)
-		(effects
-			(font
-				(size 1.27 1.27)
-			)
-			(justify left)
-		)
-	)
-	(hierarchical_label "IN1"
-		(shape input)
-		(at 109.22 85.09 180)
-		(fields_autoplaced yes)
-		(effects
-			(font
-				(size 1.27 1.27)
-			)
-			(justify right)
-		)
-	)
-	(hierarchical_label "IN2"
-		(shape input)
-		(at 109.22 87.63 180)
-		(fields_autoplaced yes)
-		(effects
-			(font
-				(size 1.27 1.27)
-			)
 			(justify right)
 		)
@@
 		(shape input)
 		(at 109.22 93.98 180)
-		(fields_autoplaced yes)
 		(effects
 			(font
@@
 		(on_board yes)
 		(dnp no)
-		(property "Reference" "#PWR088"
+		(property "Reference" "#PWR079"
 			(at 162.56 121.92 0)
 			(effects
@@
 		(on_board yes)
 		(dnp no)
-		(property "Reference" "#PWR083"
+		(property "Reference" "#PWR074"
 			(at 74.93 107.95 0)
 			(effects
@@
 		(on_board yes)
 		(dnp no)
-		(property "Reference" "#PWR090"
+		(property "Reference" "#PWR081"
 			(at 205.74 123.19 0)
 			(effects
@@
 		(on_board yes)
 		(dnp no)
-		(property "Reference" "#PWR089"
+		(property "Reference" "#PWR080"
 			(at 205.74 100.33 0)
 			(effects
@@
 		(on_board yes)
 		(dnp no)
-		(property "Reference" "#PWR087"
+		(property "Reference" "#PWR078"
 			(at 153.67 121.92 0)
 			(effects
@@
 		(on_board yes)
 		(dnp no)
-		(property "Reference" "D1"
+		(property "Reference" "D3"
 			(at 204.47 88.9 90)
 			(effects
@@
 		(on_board yes)
 		(dnp no)
-		(property "Reference" "#PWR086"
+		(property "Reference" "#PWR077"
 			(at 137.16 121.92 0)
 			(effects
@@
 		(on_board yes)
 		(dnp no)
-		(property "Reference" "#PWR084"
+		(property "Reference" "#PWR075"
 			(at 119.38 121.92 0)
 			(effects
@@
 		(on_board yes)
 		(dnp no)
-		(property "Reference" "D1"
+		(property "Reference" "D4"
 			(at 204.47 111.76 90)
 			(effects
