File: hardware/rearbox/suspension_potentiometers.kicad_sch (KiCad schematic)
At the start: 10 parts

Commit message: Changed power section
Parts:
- gave numbers to parts that had none: 6
Changed lines of the file:
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@@
 (kicad_sch
-	(version 20231120)
+	(version 20250114)
 	(generator "eeschema")
-	(generator_version "8.0")
+	(generator_version "9.0")
 	(paper "A4")
 	(title_block
@@
 		(comment 1 "Reviewer:")
 	)
+	(text "Rx\n5k"
+		(exclude_from_sim no)
+		(at 112.395 80.645 0)
+		(effects
+			(font
+				(size 1.27 1.27)
+			)
+			(justify right bottom)
+		)
+	)
+	(text "G = 2\nR_{F} = 4k7\nR_{G} = 4k7"
+		(exclude_from_sim no)
+		(at 166.37 138.43 0)
+		(effects
+			(font
+				(size 1.27 1.27)
+			)
+			(justify left bottom)
+		)
+	)
+	(text "G = 2\nR_{F} = 4k7\nR_{G} = 4k7"
+		(exclude_from_sim no)
+		(at 166.37 90.17 0)
+		(effects
+			(font
+				(size 1.27 1.27)
+			)
+			(justify left bottom)
+		)
+	)
+	(text "Rx\n5k"
+		(exclude_from_sim no)
+		(at 112.395 128.905 0)
+		(effects
+			(font
+				(size 1.27 1.27)
+			)
+			(justify right bottom)
+		)
+	)
+	(text_box "Resistance range (roughly estimated):\n1000 to 4000 Ω\n\nOptimum value of the upper resistor in the divider:\nR = sqrt(1000 * 4000) ≈ 2 kΩ\n\nOutput range:\n1.9 V to 0.238 V"
+		(exclude_from_sim no)
+		(at 33.02 35.56 0)
+		(size 39.37 22.86)
+		(margins 0.9524 0.9524 0.9524 0.9524)
+		(stroke
+			(width -0.0001)
+			(type default)
+		)
+		(fill
+			(type none)
+		)
+		(effects
+			(font
+				(size 1.27 1.27)
+			)
+			(justify left top)
+		)
+	)
 	(junction
 		(at 121.92 64.77)
@@
 		)
 	)
-	(text_box "Resistance range (roughly estimated):\n1000 to 4000 Ω\n\nOptimum value of the upper resistor in the divider:\nR = sqrt(1000 * 4000) ≈ 2 kΩ\n\nOutput range:\n1.9 V to 0.238 V"
-		(exclude_from_sim no)
-		(at 33.02 35.56 0)
-		(size 39.37 22.86)
-		(stroke
-			(width -0.0001)
-			(type default)
-		)
-		(fill
-			(type none)
-		)
+	(label "P2"
+		(at 157.48 118.11 180)
 		(effects
 			(font
 				(size 1.27 1.27)
 			)
-			(justify left top)
-		)
-	)
-	(text "Rx\n5k"
-		(exclude_from_sim no)
-		(at 112.395 80.645 0)
+			(justify right bottom)
+		)
+	)
+	(label "N2"
+		(at 119.38 121.92 180)
 		(effects
 			(font
@@
 		)
 	)
-	(text "G = 2\nR_{F} = 4k7\nR_{G} = 4k7"
-		(exclude_from_sim no)
-		(at 166.37 138.43 0)
+	(label "N1"
+		(at 119.38 73.66 180)
 		(effects
 			(font
 				(size 1.27 1.27)
 			)
-			(justify left bottom)
-		)
-	)
-	(text "G = 2\nR_{F} = 4k7\nR_{G} = 4k7"
-		(exclude_from_sim no)
-		(at 166.37 90.17 0)
+			(justify right bottom)
+		)
+	)
+	(label "P1"
+		(at 124.46 73.66 0)
 		(effects
 			(font
@@
 		)
 	)
-	(text "Rx\n5k"
-		(exclude_from_sim no)
-		(at 112.395 128.905 0)
+	(label "N2"
+		(at 153.67 124.46 180)
 		(effects
 			(font
@@
 		)
 	)
-	(label "P2"
-		(at 157.48 118.11 180)
-		(fields_autoplaced yes)
+	(label "N1"
+		(at 153.67 76.2 180)
 		(effects
 			(font
@@
 		)
 	)
-	(label "N2"
-		(at 119.38 121.92 180)
-		(fields_autoplaced yes)
+	(label "P2"
+		(at 124.46 121.92 0)
 		(effects
 			(font
 				(size 1.27 1.27)
 			)
-			(justify right bottom)
-		)
-	)
-	(label "N1"
-		(at 119.38 73.66 180)
-		(fields_autoplaced yes)
+			(justify left bottom)
+		)
+	)
+	(label "P1"
+		(at 157.48 69.85 180)
 		(effects
 			(font
@@
 		)
 	)
-	(label "P1"
-		(at 124.46 73.66 0)
-		(fields_autoplaced yes)
+	(hierarchical_label "OUT_R"
+		(shape output)
+		(at 184.15 118.11 0)
 		(effects
 			(font
 				(size 1.27 1.27)
 			)
-			(justify left bottom)
-		)
-	)
-	(label "N2"
-		(at 153.67 124.46 180)
-		(fields_autoplaced yes)
+			(justify left)
+		)
+	)
+	(hierarchical_label "OUT_L"
+		(shape output)
+		(at 184.15 69.85 0)
 		(effects
 			(font
 				(size 1.27 1.27)
 			)
-			(justify right bottom)
-		)
-	)
-	(label "N1"
-		(at 153.67 76.2 180)
-		(fields_autoplaced yes)
+			(justify left)
+		)
+	)
+	(hierarchical_label "IN_R"
+		(shape input)
+		(at 109.22 121.92 180)
 		(effects
 			(font
 				(size 1.27 1.27)
 			)
-			(justify right bottom)
-		)
-	)
-	(label "P2"
-		(at 124.46 121.92 0)
-		(fields_autoplaced yes)
-		(effects
-			(font
-				(size 1.27 1.27)
-			)
-			(justify left bottom)
-		)
-	)
-	(label "P1"
-		(at 157.48 69.85 180)
-		(fields_autoplaced yes)
-		(effects
-			(font
-				(size 1.27 1.27)
-			)
-			(justify right bottom)
-		)
-	)
-	(hierarchical_label "OUT_R"
-		(shape output)
-		(at 184.15 118.11 0)
-		(fields_autoplaced yes)
-		(effects
-			(font
-				(size 1.27 1.27)
-			)
-			(justify left)
-		)
-	)
-	(hierarchical_label "OUT_L"
-		(shape output)
-		(at 184.15 69.85 0)
-		(fields_autoplaced yes)
-		(effects
-			(font
-				(size 1.27 1.27)
-			)
-			(justify left)
-		)
-	)
-	(hierarchical_label "IN_R"
-		(shape input)
-		(at 109.22 121.92 180)
-		(fields_autoplaced yes)
-		(effects
-			(font
-				(size 1.27 1.27)
-			)
 			(justify right)
 		)
@@
 		(shape input)
 		(at 109.22 73.66 180)
-		(fields_autoplaced yes)
 		(effects
 			(font
@@
 		(on_board yes)
 		(dnp no)
-		(property "Reference" "R?"
+		(property "Reference" "R116"
 			(at 131.318 66.1416 0)
 			(effects
@@
 		(on_board yes)
 		(dnp no)
-		(property "Reference" "R?"
+		(property "Reference" "R117"
 			(at 131.318 76.3016 0)
 			(effects
@@
 		(on_board yes)
 		(dnp no)
-		(property "Reference" "#PWR?"
+		(property "Reference" "#PWR0227"
 			(at 121.92 138.43 0)
 			(effects
@@
 		(on_board yes)
 		(dnp no)
-		(property "Reference" "R?"
+		(property "Reference" "R118"
 			(at 131.318 114.4016 0)
 			(effects
@@
 		(on_board yes)
 		(dnp no)
-		(property "Reference" "R?"
+		(property "Reference" "R115"
 			(at 112.522 114.4016 0)
 			(effects
@@
 		(on_board yes)
 		(dnp no)
-		(property "Reference" "#PWR?"
+		(property "Reference" "#PWR0225"
 			(at 121.92 90.17 0)
 			(effects
@@
 		(on_board yes)
 		(dnp no)
-		(property "Reference" "R?"
+		(property "Reference" "R114"
 			(at 112.522 66.1416 0)
 			(effects
@@
 		(on_board yes)
 		(dnp no)
-		(property "Reference" "R?"
+		(property "Reference" "R119"
 			(at 131.318 124.5616 0)
 			(effects
@@
 		(at 158.75 114.3)
 		(size 24.13 13.97)
+		(exclude_from_sim no)
+		(in_bom yes)
+		(on_board yes)
+		(dnp no)
 		(stroke
 			(width 0.1524)
@@
 		(at 158.75 66.04)
 		(size 24.13 13.97)
+		(exclude_from_sim no)
+		(in_bom yes)
+		(on_board yes)
+		(dnp no)
 		(stroke
 			(width 0.1524)
