File: hardware/rearbox/assi.kicad_sch (KiCad schematic)
At the start: 16 parts, among them Q2 BUK6D210, Q3 BUK6D210, Q4 BUK6D210, Q5 BUK6D210

Commit message: Changed power section
Parts:
- gave numbers to parts that had none: 7
Changed lines of the file:
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@@
 (kicad_sch
-	(version 20231120)
+	(version 20250114)
 	(generator "eeschema")
-	(generator_version "8.0")
+	(generator_version "9.0")
 	(paper "A4")
 	(title_block
@@
 		(comment 1 "Reviewer:")
 	)
+	(text "+24V"
+		(exclude_from_sim no)
+		(at 131.9784 77.1906 0)
+		(effects
+			(font
+				(size 1.27 1.27)
+			)
+			(justify left bottom)
+		)
+	)
+	(text "+24V"
+		(exclude_from_sim no)
+		(at 260.2484 84.8106 0)
+		(effects
+			(font
+				(size 1.27 1.27)
+			)
+			(justify left bottom)
+		)
+	)
+	(text "Red Channel"
+		(exclude_from_sim no)
+		(at 75.565 97.536 90)
+		(effects
+			(font
+				(size 1.27 1.27)
+			)
+			(justify left bottom)
+		)
+	)
+	(text "+24V"
+		(exclude_from_sim no)
+		(at 72.2884 78.3844 0)
+		(effects
+			(font
+				(size 1.27 1.27)
+			)
+			(justify left bottom)
+		)
+	)
+	(text "+24V"
+		(exclude_from_sim no)
+		(at 191.643 78.359 0)
+		(effects
+			(font
+				(size 1.27 1.27)
+			)
+			(justify left bottom)
+		)
+	)
+	(text "Blue Channel"
+		(exclude_from_sim no)
+		(at 194.945 97.536 90)
+		(effects
+			(font
+				(size 1.27 1.27)
+			)
+			(justify left bottom)
+		)
+	)
+	(text "Green Channel"
+		(exclude_from_sim no)
+		(at 135.255 97.536 90)
+		(effects
+			(font
+				(size 1.27 1.27)
+			)
+			(justify left bottom)
+		)
+	)
+	(text "Buzzer"
+		(exclude_from_sim no)
+		(at 263.525 97.536 90)
+		(effects
+			(font
+				(size 1.27 1.27)
+			)
+			(justify left bottom)
+		)
+	)
 	(junction
 		(at 106.68 107.95)
@@
 		)
 	)
-	(text "+24V"
-		(exclude_from_sim no)
-		(at 131.9784 77.1906 0)
+	(hierarchical_label "IN_BUZZER"
+		(shape input)
+		(at 219.71 107.95 180)
 		(effects
 			(font
 				(size 1.27 1.27)
 			)
-			(justify left bottom)
-		)
-	)
-	(text "+24V"
-		(exclude_from_sim no)
-		(at 260.2484 84.8106 0)
+			(justify right)
+		)
+	)
+	(hierarchical_label "IN_G"
+		(shape input)
+		(at 96.52 107.95 180)
 		(effects
 			(font
 				(size 1.27 1.27)
 			)
-			(justify left bottom)
-		)
-	)
-	(text "Red Channel"
-		(exclude_from_sim no)
-		(at 75.565 97.536 90)
+			(justify right)
+		)
+	)
+	(hierarchical_label "OUT_G"
+		(shape output)
+		(at 119.38 100.33 0)
 		(effects
 			(font
 				(size 1.27 1.27)
 			)
-			(justify left bottom)
-		)
-	)
-	(text "+24V"
-		(exclude_from_sim no)
-		(at 72.2884 78.3844 0)
+			(justify left)
+		)
+	)
+	(hierarchical_label "IN_R"
+		(shape input)
+		(at 36.83 107.95 180)
 		(effects
 			(font
 				(size 1.27 1.27)
 			)
-			(justify left bottom)
-		)
-	)
-	(text "+24V"
-		(exclude_from_sim no)
-		(at 191.643 78.359 0)
+			(justify right)
+		)
+	)
+	(hierarchical_label "OUT_R"
+		(shape output)
+		(at 59.69 100.33 0)
 		(effects
 			(font
 				(size 1.27 1.27)
 			)
-			(justify left bottom)
-		)
-	)
-	(text "Blue Channel"
-		(exclude_from_sim no)
-		(at 194.945 97.536 90)
+			(justify left)
+		)
+	)
+	(hierarchical_label "OUT_BUZZER"
+		(shape output)
+		(at 242.57 100.33 0)
 		(effects
 			(font
 				(size 1.27 1.27)
 			)
-			(justify left bottom)
-		)
-	)
-	(text "Green Channel"
-		(exclude_from_sim no)
-		(at 135.255 97.536 90)
+			(justify left)
+		)
+	)
+	(hierarchical_label "IN_B"
+		(shape input)
+		(at 156.21 107.95 180)
 		(effects
 			(font
 				(size 1.27 1.27)
 			)
-			(justify left bottom)
-		)
-	)
-	(text "Buzzer"
-		(exclude_from_sim no)
-		(at 263.525 97.536 90)
-		(effects
-			(font
-				(size 1.27 1.27)
-			)
-			(justify left bottom)
-		)
-	)
-	(hierarchical_label "IN_BUZZER"
-		(shape input)
-		(at 219.71 107.95 180)
-		(fields_autoplaced yes)
-		(effects
-			(font
-				(size 1.27 1.27)
-			)
-			(justify right)
-		)
-	)
-	(hierarchical_label "IN_G"
-		(shape input)
-		(at 96.52 107.95 180)
-		(fields_autoplaced yes)
-		(effects
-			(font
-				(size 1.27 1.27)
-			)
-			(justify right)
-		)
-	)
-	(hierarchical_label "OUT_G"
-		(shape output)
-		(at 119.38 100.33 0)
-		(fields_autoplaced yes)
-		(effects
-			(font
-				(size 1.27 1.27)
-			)
-			(justify left)
-		)
-	)
-	(hierarchical_label "IN_R"
-		(shape input)
-		(at 36.83 107.95 180)
-		(fields_autoplaced yes)
-		(effects
-			(font
-				(size 1.27 1.27)
-			)
-			(justify right)
-		)
-	)
-	(hierarchical_label "OUT_R"
-		(shape output)
-		(at 59.69 100.33 0)
-		(fields_autoplaced yes)
-		(effects
-			(font
-				(size 1.27 1.27)
-			)
-			(justify left)
-		)
-	)
-	(hierarchical_label "OUT_BUZZER"
-		(shape output)
-		(at 242.57 100.33 0)
-		(fields_autoplaced yes)
-		(effects
-			(font
-				(size 1.27 1.27)
-			)
-			(justify left)
-		)
-	)
-	(hierarchical_label "IN_B"
-		(shape input)
-		(at 156.21 107.95 180)
-		(fields_autoplaced yes)
-		(effects
-			(font
-				(size 1.27 1.27)
-			)
 			(justify right)
 		)
@@
 		(shape output)
 		(at 179.07 100.33 0)
-		(fields_autoplaced yes)
 		(effects
 			(font
@@
 		(on_board yes)
 		(dnp no)
-		(property "Reference" "R?"
+		(property "Reference" "R30"
 			(at 171.45 113.03 90)
 			(effects
@@
 		(on_board yes)
 		(dnp no)
-		(property "Reference" "R?"
+		(property "Reference" "R29"
 			(at 161.29 105.41 90)
 			(effects
@@
 		(on_board yes)
 		(dnp no)
-		(property "Reference" "R?"
+		(property "Reference" "R26"
 			(at 52.07 113.03 90)
 			(effects
@@
 		(on_board yes)
 		(dnp no)
-		(property "Reference" "R?"
+		(property "Reference" "R28"
 			(at 111.76 113.03 90)
 			(effects
@@
 		(on_board yes)
 		(dnp no)
-		(property "Reference" "R?"
+		(property "Reference" "R25"
 			(at 41.91 105.41 90)
 			(effects
@@
 		(on_board yes)
 		(dnp no)
-		(property "Reference" "R?"
+		(property "Reference" "R32"
 			(at 234.95 113.03 90)
 			(effects
@@
 		(on_board yes)
 		(dnp no)
-		(property "Reference" "R?"
+		(property "Reference" "R27"
 			(at 101.6 105.41 90)
 			(effects

Commit message: Sync :(
Other:
- note added: "30.07.2025 Currently used as brake light transtor"
Changed lines of the file:
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@@
+		)
+	)
+	(text "30.07.2025\nCurrently used as brake light transtor\n"
+		(exclude_from_sim no)
+		(at 172.974 92.964 0)
+		(effects
+			(font
+				(size 1.27 1.27)
+			)
 		)
 	)
